File: kicad/ant_weight.sch (KiCad schematic (older format))
At the start: 63 parts, among them J1 BATT_JST, J10 Pi Header, J11 FR, J12 RW, J13 FW, J14 3V3 Only, J2 GS3, J3 I2C, J4 FTDI, J5 GS3, J6 SBus Rx, J7 RL, J8 FL, J9 RR, SW1 POWER, SW2 RESET, SW3 PROGRAM, U1 BA50DD0WHFP, U10 WS2812B, U11 WS2812B, U2 BA33DD0WHFP, U3 XBee, U4 ESP32-WROOM, U5 BD622xxx, U6 BD622xxx, U7 BD622xxx, U8 WS2812B, U9 WS2812B

Commit message: Upgraded to kicad v5
Parts:
- C1, C11, C12, C13, C14, C3, C5, C6, C7: symbol C -> Device:C
- C10, C8, C9: symbol CP1_Small -> Device:CP1_Small
- C2, C4: symbol CP -> Device:CP
- D1, D2: symbol D_Schottky -> Device:D_Schottky
- D3, D4, D5, D6, D7, D8: symbol LED -> Device:LED
- J1, J11, J12, J13, J14, J7, J8, J9: symbol Conn_01x02 -> ant_weight-rescue:Conn_01x02
- J10: symbol Conn_02x20_Odd_Even -> ant_weight-rescue:Conn_02x20_Odd_Even
- J2, J5: symbol GS3 -> ant_weight-rescue:GS3
- J3: symbol Conn_01x04 -> ant_weight-rescue:Conn_01x04
- J4: symbol Conn_01x06 -> ant_weight-rescue:Conn_01x06
- J6: symbol Conn_01x03 -> ant_weight-rescue:Conn_01x03
- R1, R10, R11, R12, R13, R2, R3, R4, R5, R6, R7, R8, R9: symbol R -> Device:R
- SW1: symbol SW_SPDT_MSM -> ant_weight-rescue:SW_SPDT_MSM
- SW2, SW3: symbol SW_Push -> ant_weight-rescue:SW_Push
- U1, U2: symbol BA33DD0WHFP -> BA33DD0WHFP_Regulator:BA33DD0WHFP
- U10, U11, U8, U9: symbol WS2812B -> ws2812b:WS2812B
- U3: symbol XBee -> xbee:XBee
- U4: symbol ESP32-WROOM -> ESP32-footprints-Shem-Lib:ESP32-WROOM
- U5, U6, U7: symbol BD622xxx -> bd622xxx_HBridge:BD622xxx
